File: P.I6Def/P.I6Def.kicad_sch (KiCad schematic)
At the start: 41 parts, among them J1 B3B-PH-K-S, J2 B3B-PH-K-S, J3 CX90B-16P1, J4 B4B-PH-SM4-TB_LF__SN__P_, J5 B4B-PH-SM4-TB_LF__SN__P_, SW2 SW_SPST, SW3 SW_SPST, U2 LMV321IDCKT, U3 LMV321IDCKT, U4 LMV321IDCKT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

Commit message: MEJORA DE LA PCB
Parts:
- removed X1: ESP32-S3-WROOM-1-N16R8, ESP32-S3-WROOM-1-N16R8:ESP32S3WROOM1N8R2, symbol ESP32-S3-WROOM-1-N16R8:ESP32-S3-WROOM-1-N16R8
- added U6: ESP32-S3-WROOM-1, RF_Module:ESP32-S3-WROOM-1U, symbol RF_Module:ESP32-S3-WROOM-1
Connections:
- net VBUS_B is gone; now on net +5V: C1.1, C2.1, J3.B4 (VBUS_B), J3.B9 (VBUS_B), VR1.1 (EN), VR1.4 (IN)
- net +3.3V: now also U6.2 (3V3)
- net ADC1_CH0: now also U6.5 (IO5)
- net ADC1_CH1: now also U6.4 (IO4)
- net ADDR_CCS811: now also U6.35 (IO42)
- net D+: now also U6.14 (USB_D+)
- net D-: now also U6.13 (USB_D-)
- net GND: now also U6.1 (GND), U6.40 (GND), U6.41 (GND)
- net SCL_CSS811: now also U6.32 (IO39)
- net SDA_CSS811: now also U6.31 (IO38)
- net WAKE_CCS811: now also U6.33 (IO40)
- net nINT_CCS811: now also U6.34 (IO41)
- net BOOT: now reaches C9.1, R8.1, SW3.1 (A)
- net BOOT: now also U6.27 (IO0)
- net at C6.1, R7.2, SW2.1 (A): now also U6.3 (EN)
- no-connect marks 31 -> 27
Other:
- moved on the sheet: C11, C12, C14, C15, C16, C17, C5, C6, C7, C8, C9, J1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

Commit message: Actualizacion PCB
Connections:
- net ADC1_CH0: now also U6.17 (IO9); no longer U6.5 (IO5)
- net ADC1_CH1: now also U6.18 (IO10); no longer U6.4 (IO4)
- no-connect marks 27 -> 25

Commit message: Actualizacion PCB
Parts:
- added R14: 4.7k, ERA6AEB472V:RES_ERA6AEB472V, symbol Device:R
- C16: value 0.1u -> 1uF; footprint C0805C104K8RACTU:CAPC2012X88N -> C2012X5R1C105K085AA:CAPC2012X100N
- R11: value 10k -> 4.7k; footprint MCU08050C1002FP500:RESC2012X55N -> ERA6AEB472V:RES_ERA6AEB472V
Connections:
- net +3.3V: now also R14.1
- net nINT_CCS811: now also R14.2
- no-connect marks 25 -> 29
Other:
- moved on the sheet: C15, C17, C7, J2, R4, R5, R6, U3, U4
